Commit message: applied rotation to link3

File: synriard/urdf/Alicia_D_v5_6/Alicia_D_v5_6_leader_ur.urdf (robot description, URDF)
Before this commit: robot Alicia_D_v5_6_leader_ur, 8 links, 7 joints
Joints:
- joint joint3: origin xyz=0.18922 0.027473 -0.00041 rpy=0 0 0.7854 -> xyz=0.18922 0.027473 -0.00041 rpy=0 3.14159 0.7854

Commit message: updated joint3 motion range

File: synriard/urdf/Alicia_D_v5_6/Alicia_D_v5_6_leader_ur.urdf (robot description, URDF)
Before this commit: robot Alicia_D_v5_6_leader_ur, 8 links, 7 joints
Joints:
- joint joint3: axis 0 0 -1 -> 0 0 1; limit lower=0.6 upper=2.2 effort=5 velocity=12 -> lower=-0.6 upper=2.2 effort=5 velocity=12
